File: kicad/hackpad-san.kicad_pcb (KiCad board)
At the start: 2 copper layers, 115.5 x 73 mm, 24 parts, among them SW1 SW_Push, SW11 RotaryEncoder_Switch, SW2 SW_Push, SW3 SW_Push, SW4 SW_Push, SW5 SW_Push, SW6 SW_Push, SW7 SW_Push, SW8 SW_Push, SW9 SW_Push, U1 XIAO-RP2040-SMD

Commit message: added
Connections:
- U1 pad 7: unconnected-(U1-D6-Pad7) -> /RE_A
- U1 pad 8: unconnected-(U1-D7-Pad8) -> /RE_B
- U1 pad 9: unconnected-(U1-D8-Pad9) -> /RE_S1
Routing:
- net /RE_B: track 0.00 -> 112.9 mm, vias 0 -> 2
- net /RE_S1: track 0.00 -> 106.7 mm, vias 0 -> 2
- net /RE_A: track 0.00 -> 93.2 mm, vias 0 -> 2
