File: kicad/hackpad-san.kicad_sch (KiCad schematic)
At the start: 24 parts, among them SW1 SW_Push, SW11 RotaryEncoder_Switch, SW2 SW_Push, SW3 SW_Push, SW4 SW_Push, SW5 SW_Push, SW6 SW_Push, SW7 SW_Push, SW8 SW_Push, SW9 SW_Push, U1 XIAO-RP2040-SMD

Commit message: added
Connections:
- net RE_A: now also U1.7 (D6)
- net RE_B: now also U1.8 (D7)
- net RE_S1: now also U1.9 (D8)
Changed lines of the file:
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@@
+	(wire
+		(pts
+			(xy 243.84 82.55) (xy 237.49 82.55)
+		)
+		(stroke
+			(width 0)
+			(type default)
+		)
+	)
 	(wire
 		(pts
@@
 	(wire
 		(pts
+			(xy 187.96 86.36) (xy 194.31 86.36)
+		)
+		(stroke
+			(width 0)
+			(type default)
+		)
+	)
+	(wire
+		(pts
 			(xy 148.59 109.22) (xy 157.48 109.22)
 		)
@@
 		(pts
 			(xy 138.43 43.18) (xy 138.43 59.69)
+		)
+		(stroke
+			(width 0)
+			(type default)
+		)
+	)
+	(wire
+		(pts
+			(xy 237.49 86.36) (xy 242.57 86.36)
 		)
 		(stroke
@@
 		)
 	)
+	(label "RE_A"
+		(at 187.96 86.36 0)
+		(effects
+			(font
+				(size 1.27 1.27)
+			)
+			(justify left bottom)
+		)
+	)
 	(label "row3"
 		(at 138.43 43.18 0)
@@
 		)
 	)
+	(label "RE_B"
+		(at 242.57 86.36 0)
+		(effects
+			(font
+				(size 1.27 1.27)
+			)
+			(justify left bottom)
+		)
+	)
 	(label "col1"
 		(at 186.69 74.93 0)
@@
 		(effects
 			(font
+				(size 1.27 1.27)
+			)
+			(justify left bottom)
+		)
+	)
+	(label "RE_S1"
+		(at 243.84 82.55 0)
+		(effects
+			(font
